Commit message: Make joint7 initial position compatible with franka_description

File: urdf/panda.urdf (robot description, URDF)
Before this commit: robot panda, 12 links, 11 joints
Joints:
- joint panda_hand_joint: origin xyz=0 0 0.107 rpy=0 0 0 -> xyz=0 0 0.107 rpy=0 0 -0.7853981633974483

Commit message: Remove obselete inertial properties from URDF
Signed-off-by: Andrej Orsula <orsula.andrej@gmail.com>

File: urdf/panda.urdf (robot description, URDF)
Before this commit: robot panda, 12 links, 11 joints
Links:
- link panda_hand: mass 0.73 -> None
- link panda_leftfinger: mass 0.1 -> None
- link panda_link0: mass 2.92 -> None
- link panda_link1: mass 2.74 -> None
- link panda_link2: mass 2.74 -> None
- link panda_link3: mass 2.38 -> None
- link panda_link4: mass 2.38 -> None
- link panda_link5: mass 2.74 -> None
- link panda_link6: mass 1.55 -> None
- link panda_link7: mass 0.54 -> None
- link panda_rightfinger: mass 0.1 -> None
