Commit message: Add xacro-based URDF and SDF (with ros2_control)
Signed-off-by: Andrej Orsula <orsula.andrej@gmail.com>

File: panda_description/urdf/panda_arm.xacro (robot description, xacro)
@@ -1,313 +1,348 @@
-<?xml version='1.0' encoding='utf-8'?>
-<robot xmlns:xacro="http://www.ros.org/wiki/xacro" name="panda">
-  <!-- safety_distance: Minimum safety distance in [m] by which the collision volumes are expanded and which is enforced during robot motions -->
-  <!-- arm_id: Namespace of the panda arm. Serves to differentiate between arms in case of multiple instances. -->
-  <xacro:macro name="panda_arm" params="arm_id:='panda' description_pkg:='franka_description' connected_to:='' xyz:='0 0 0' rpy:='0 0 0' safety_distance:=0">
-    <xacro:unless value="${not connected_to}">
-      <joint name="${arm_id}_joint_${connected_to}" type="fixed">
-        <parent link="${connected_to}"/>
-        <child link="${arm_id}_link0"/>
-        <origin rpy="${rpy}" xyz="${xyz}"/>
-      </joint>
-    </xacro:unless>
-    <link name="${arm_id}_link0">
-      <visual>
-        <geometry>
-          <mesh filename="package://${description_pkg}/meshes/visual/link0.dae"/>
-        </geometry>
-      </visual>
-      <collision>
-        <origin xyz="-0.075 0 0.06" rpy="0 ${pi/2} 0"/>
-        <geometry>
-          <cylinder radius="${0.06+safety_distance}" length="0.03" />
-        </geometry>
-      </collision>
-      <collision>
-        <origin xyz="-0.06 0 0.06" rpy="0 0 0"/>
-        <geometry>
-          <sphere radius="${0.06+safety_distance}" />
-        </geometry>
-      </collision>
-      <collision>
-        <origin xyz="-0.09 0 0.06" rpy="0 0 0"/>
-        <geometry>
-          <sphere radius="${0.06+safety_distance}" />
-        </geometry>
-      </collision>
-    </link>
-    <link name="${arm_id}_link1">
-      <visual>
-        <geometry>
-          <mesh filename="package://${description_pkg}/meshes/visual/link1.dae"/>
-        </geometry>
-      </visual>
-      <collision>
-        <origin xyz="0 0 -0.1915" rpy="0 0 0"/>
-        <geometry>
-          <cylinder radius="${0.06+safety_distance}" length="0.2830" />
-        </geometry>
-      </collision>
-      <collision>
-        <origin xyz="0 0 -0.333" rpy="0 0 0"/>
-        <geometry>
-          <sphere radius="${0.06+safety_distance}" />
-        </geometry>
-      </collision>
-      <collision>
-        <origin xyz="0 0 -0.05" rpy="0 0 0"/>
-        <geometry>
-          <sphere radius="${0.06+safety_distance}" />
-        </geometry>
-      </collision>
-    </link>
-    <joint name="${arm_id}_joint1" type="revolute">
-      <safety_controller k_position="100.0" k_velocity="40.0" soft_lower_limit="-2.8973" soft_upper_limit="2.8973"/>
-      <origin rpy="0 0 0" xyz="0 0 0.333"/>
-      <parent link="${arm_id}_link0"/>
-      <child link="${arm_id}_link1"/>
-      <axis xyz="0 0 1"/>
-      <limit effort="87" lower="-2.8973" upper="2.8973" velocity="2.1750"/>
-    </joint>
-    <link name="${arm_id}_link2">
-      <visual>
-        <geometry>
-          <mesh filename="package://${description_pkg}/meshes/visual/link2.dae"/>
-        </geometry>
-      </visual>
-      <collision>
-        <origin xyz="0 0 0" rpy="0 0 0"/>
-        <geometry>
-          <cylinder radius="${0.06+safety_distance}" length="0.12" />
-        </geometry>
-      </collision>
-      <collision>
-        <origin xyz="0 0 -0.06" rpy="0 0 0"/>
-        <geometry>
-          <sphere radius="${0.06+safety_distance}" />
-        </geometry>
-      </collision>
-      <collision>
-        <origin xyz="0 0 0.06" rpy="0 0 0"/>
-        <geometry>
-          <sphere radius="${0.06+safety_distance}" />
-        </geometry>
-      </collision>
-    </link>
-    <joint name="${arm_id}_joint2" type="revolute">
-      <safety_controller k_position="100.0" k_velocity="40.0" soft_lower_limit="-1.7628" soft_upper_limit="1.7628"/>
-      <origin rpy="${-pi/2} 0 0" xyz="0 0 0"/>
-      <parent link="${arm_id}_link1"/>
-      <child link="${arm_id}_link2"/>
-      <axis xyz="0 0 1"/>
-      <limit effort="87" lower="-1.7628" upper="1.7628" velocity="2.1750"/>
-    </joint>
-    <link name="${arm_id}_link3">
-      <visual>
-        <geometry>
-          <mesh filename="package://${description_pkg}/meshes/visual/link3.dae"/>
-        </geometry>
-      </visual>
-      <collision>
-        <origin xyz="0 0 -0.145" rpy="0 0 0"/>
-        <geometry>
-          <cylinder radius="${0.06+safety_distance}" length="0.15" />
-        </geometry>
-      </collision>
-      <collision>
-        <origin xyz="0 0 -0.22" rpy="0 0 0"/>
-        <geometry>
-          <sphere radius="${0.06+safety_distance}" />
-        </geometry>
-      </collision>
-      <collision>
-        <origin xyz="0 0 -0.07" rpy="0 0 0"/>
-        <geometry>
-          <sphere radius="${0.06+safety_distance}" />
-        </geometry>
-      </collision>
-    </link>
-    <joint name="${arm_id}_joint3" type="revolute">
-      <safety_controller k_position="100.0" k_velocity="40.0" soft_lower_limit="-2.8973" soft_upper_limit="2.8973"/>
-      <origin rpy="${pi/2} 0 0" xyz="0 -0.316 0"/>
-      <parent link="${arm_id}_link2"/>
-      <child link="${arm_id}_link3"/>
-      <axis xyz="0 0 1"/>
-      <limit effort="87" lower="-2.8973" upper="2.8973" velocity="2.1750"/>
-    </joint>
-    <link name="${arm_id}_link4">
-      <visual>
-        <geometry>
-          <mesh filename="package://${description_pkg}/meshes/visual/link4.dae"/>
-        </geometry>
-      </visual>
-      <collision>
-        <origin xyz="0 0 0" rpy="0 0 0"/>
-        <geometry>
-          <cylinder radius="${0.06+safety_distance}" length="0.12" />
-        </geometry>
-      </collision>
-      <collision>
-        <origin xyz="0 0 0.06" rpy="0 0 0"/>
-        <geometry>
-          <sphere radius="${0.06+safety_distance}" />
-        </geometry>
-      </collision>
-      <collision>
-        <origin xyz="0 0 -0.06" rpy="0 0 0"/>
-        <geometry>
-          <sphere radius="${0.06+safety_distance}" />
-        </geometry>
-      </collision>
-    </link>
-    <joint name="${arm_id}_joint4" type="revolute">
-      <safety_controller k_position="100.0" k_velocity="40.0" soft_lower_limit="-3.0718" soft_upper_limit="-0.0698"/>
-      <origin rpy="${pi/2} 0 0" xyz="0.0825 0 0"/>
-      <parent link="${arm_id}_link3"/>
-      <child link="${arm_id}_link4"/>
-      <axis xyz="0 0 1"/>
-      <limit effort="87" lower="-3.0718" upper="-0.0698" velocity="2.1750"/>
-    </joint>
-    <link name="${arm_id}_link5">
-      <visual>
-        <geometry>
-          <mesh filename="package://${description_pkg}/meshes/visual/link5.dae"/>
-        </geometry>
-      </visual>
-      <collision>
-        <origin xyz="0 0 -0.26" rpy="0 0 0"/>
-        <geometry>
-          <cylinder radius="${0.06+safety_distance}" length="0.1" />
-        </geometry>
-      </collision>
-      <collision>
-        <origin xyz="0 0 -0.31" rpy="0 0 0"/>
-        <geometry>
-          <sphere radius="${0.06+safety_distance}" />
-        </geometry>
-      </collision>
-      <collision>
-        <origin xyz="0 0 -0.21" rpy="0 0 0"/>
-        <geometry>
-          <sphere radius="${0.06+safety_distance}" />
-        </geometry>
-      </collision>
-      <collision>
-        <origin xyz="0 0.08 -0.13" rpy="0 0 0"/>
-        <geometry>
-          <cylinder radius="${0.025+safety_distance}" length="0.14" />
-        </geometry>
-      </collision>
-      <collision>
-        <origin xyz="0 0.08 -0.06" rpy="0 0 0"/>
-        <geometry>
-          <sphere radius="${0.025+safety_distance}" />
-        </geometry>
-      </collision>
-      <collision>
-        <origin xyz="0 0.08 -0.20" rpy="0 0 0"/>
-        <geometry>
-          <sphere radius="${0.025+safety_distance}" />
-        </geometry>
-      </collision>
-    </link>
-    <joint name="${arm_id}_joint5" type="revolute">
-      <safety_controller k_position="100.0" k_velocity="40.0" soft_lower_limit="-2.8973" soft_upper_limit="2.8973"/>
-      <origin rpy="${-pi/2} 0 0" xyz="-0.0825 0.384 0"/>
-      <parent link="${arm_id}_link4"/>
-      <child link="${arm_id}_link5"/>
-      <axis xyz="0 0 1"/>
-      <limit effort="12" lower="-2.8973" upper="2.8973" velocity="2.6100"/>
-    </joint>
-    <link name="${arm_id}_link6">
-      <visual>
-        <geometry>
-          <mesh filename="package://${description_pkg}/meshes/visual/link6.dae"/>
-        </geometry>
-      </visual>
-      <collision>
-        <origin xyz="0 0 -0.03" rpy="0 0 0"/>
-        <geometry>
-          <cylinder radius="${0.05+safety_distance}" length="0.08" />
-        </geometry>
-      </collision>
-      <collision>
-        <origin xyz="0 0 0.01" rpy="0 0 0"/>
-        <geometry>
-          <sphere radius="${0.05+safety_distance}" />
-        </geometry>
-      </collision>
-      <collision>
-        <origin xyz="0 0 -0.07" rpy="0 0 0"/>
-        <geometry>
-          <sphere radius="${0.05+safety_distance}" />
-        </geometry>
-      </collision>
-    </link>
-    <joint name="${arm_id}_joint6" type="revolute">
-      <safety_controller k_position="100.0" k_velocity="40.0" soft_lower_limit="-0.0175" soft_upper_limit="3.7525"/>
-      <origin rpy="${pi/2} 0 0" xyz="0 0 0"/>
-      <parent link="${arm_id}_link5"/>
-      <child link="${arm_id}_link6"/>
-      <axis xyz="0 0 1"/>
-      <limit effort="12" lower="-0.0175" upper="3.7525" velocity="2.6100"/>
-    </joint>
-    <link name="${arm_id}_link7">
-      <visual>
-        <geometry>
-          <mesh filename="package://${description_pkg}/meshes/visual/link7.dae"/>
-        </geometry>
-      </visual>
-      <collision>
-        <origin xyz="0 0 0.01" rpy="0 0 0"/>
-        <geometry>
-          <cylinder radius="${0.04+safety_distance}" length="0.14" />
-        </geometry>
-      </collision>
-      <collision>
-        <origin xyz="0 0 0.08" rpy="0 0 0"/>
-        <geometry>
-          <sphere radius="${0.04+safety_distance}"  />
-        </geometry>
-      </collision>
-      <collision>
-        <origin xyz="0 0 -0.06" rpy="0 0 0"/>
-        <geometry>
-          <sphere radius="${0.04+safety_distance}"  />
-        </geometry>
-      </collision>
-    </link>
-    <joint name="${arm_id}_joint7" type="revolute">
-      <safety_controller k_position="100.0" k_velocity="40.0" soft_lower_limit="-2.8973" soft_upper_limit="2.8973"/>
-      <origin rpy="${pi/2} 0 0" xyz="0.088 0 0"/>
-      <parent link="${arm_id}_link6"/>
-      <child link="${arm_id}_link7"/>
-      <axis xyz="0 0 1"/>
-      <limit effort="12" lower="-2.8973" upper="2.8973" velocity="2.6100"/>
-    </joint>
-    <link name="${arm_id}_link8">
-      <collision>
-        <origin xyz="0.0424 0.0424 -0.0250" rpy="${pi} ${pi/2} ${pi/2}"/>
-        <geometry>
-          <cylinder radius="${0.03+safety_distance}"  length="0.01" />
-        </geometry>
-      </collision>
-      <collision>
-        <origin xyz="0.0424 0.0424 -0.02" rpy="0 0 0"/>
-        <geometry>
-          <sphere radius="${0.03+safety_distance}"  />
-        </geometry>
-      </collision>
-      <collision>
-        <origin xyz="0.0424 0.0424 -0.03" rpy="0 0 0"/>
-        <geometry>
-          <sphere radius="${0.03+safety_distance}"  />
-        </geometry>
-      </collision>
-    </link>
-    <joint name="${arm_id}_joint8" type="fixed">
-      <origin rpy="0 0 0" xyz="0 0 0.107"/>
-      <parent link="${arm_id}_link7"/>
-      <child link="${arm_id}_link8"/>
-    </joint>
+<?xml version="1.0"?>
+<!-- Xacro for Franka Emika Panda arm -->
+<robot xmlns:xacro="http://www.ros.org/wiki/xacro">
+  <!--                   -->
+  <!-- Imported elements -->
+  <!--                   -->
+  <xacro:include filename="$(find panda_description)/urdf/panda_utils.xacro"/>
+  <xacro:include filename="$(find panda_description)/urdf/panda.ros2_control"/>
+  <!--            -->
+  <!-- Properties -->
+  <!--            -->
+  <xacro:property name="joint_base_name" value="joint_base"/>
+  <xacro:property name="joint_base_type" value="fixed"/>
+  <xacro:property name="link0_name" value="link0"/>
+  <xacro:property name="link0_mu" value="0.85"/>
+  <xacro:property name="joint1_name" value="joint1"/>
+  <xacro:property name="joint1_type" value="revolute"/>
+  <xacro:property name="joint1_origin_xyz" value="0 0 0.333"/>
+  <xacro:property name="joint1_origin_rpy" value="0 0 0"/>
+  <xacro:property name="joint1_axis_xyz" value="0 0 1"/>
+  <xacro:property name="joint1_lower_limit" value="${-166*pi/180}"/>
+  <xacro:property name="joint1_upper_limit" value="${166*pi/180}"/>
+  <xacro:property name="joint1_velocity_limit" value="${150*pi/180}"/>
+  <xacro:property name="joint1_torque_limit" value="87"/>
+  <xacro:property name="joint1_damping" value="21.75"/>
+  <xacro:property name="joint1_friction" value="3.48"/>
+  <xacro:property name="link1_name" value="link1"/>
+  <xacro:property name="link1_mu" value="0.85"/>
+  <xacro:property name="joint2_name" value="joint2"/>
+  <xacro:property name="joint2_type" value="revolute"/>
+  <xacro:property name="joint2_origin_xyz" value="0 0 0"/>
+  <xacro:property name="joint2_origin_rpy" value="${-pi/2} 0 0"/>
+  <xacro:property name="joint2_axis_xyz" value="0 0 1"/>
+  <xacro:property name="joint2_lower_limit" value="${-101*pi/180}"/>
+  <xacro:property name="joint2_upper_limit" value="${101*pi/180}"/>
+  <xacro:property name="joint2_velocity_limit" value="${150*pi/180}"/>
+  <xacro:property name="joint2_torque_limit" value="87"/>
+  <xacro:property name="joint2_damping" value="21.75"/>
+  <xacro:property name="joint2_friction" value="3.48"/>
+  <xacro:property name="link2_name" value="link2"/>
+  <xacro:property name="link2_mu" value="0.85"/>
+  <xacro:property name="joint3_name" value="joint3"/>
+  <xacro:property name="joint3_type" value="revolute"/>
+  <xacro:property name="joint3_origin_xyz" value="0 -0.316 0"/>
+  <xacro:property name="joint3_origin_rpy" value="${pi/2} 0 0"/>
+  <xacro:property name="joint3_axis_xyz" value="0 0 1"/>
+  <xacro:property name="joint3_lower_limit" value="${-166*pi/180}"/>
+  <xacro:property name="joint3_upper_limit" value="${166*pi/180}"/>
+  <xacro:property name="joint3_velocity_limit" value="${150*pi/180}"/>
+  <xacro:property name="joint3_torque_limit" value="87"/>
+  <xacro:property name="joint3_damping" value="21.75"/>
+  <xacro:property name="joint3_friction" value="3.48"/>
+  <xacro:property name="link3_name" value="link3"/>
+  <xacro:property name="link3_mu" value="0.85"/>
+  <xacro:property name="joint4_name" value="joint4"/>
+  <xacro:property name="joint4_type" value="revolute"/>
+  <xacro:property name="joint4_origin_xyz" value="0.0825 0 0"/>
+  <xacro:property name="joint4_origin_rpy" value="${pi/2} 0 0"/>
+  <xacro:property name="joint4_axis_xyz" value="0 0 1"/>
+  <xacro:property name="joint4_lower_limit" value="${-176/180*pi}"/>
+  <xacro:property name="joint4_upper_limit" value="${-4/180*pi}"/>
+  <xacro:property name="joint4_velocity_limit" value="${150*pi/180}"/>
+  <xacro:property name="joint4_torque_limit" value="87"/>
+  <xacro:property name="joint4_damping" value="21.75"/>
+  <xacro:property name="joint4_friction" value="3.48"/>
+  <xacro:property name="link4_name" value="link4"/>
+  <xacro:property name="link4_mu" value="0.85"/>
+  <xacro:property name="joint5_name" value="joint5"/>
+  <xacro:property name="joint5_type" value="revolute"/>
+  <xacro:property name="joint5_origin_xyz" value="-0.0825 0.384 0"/>
+  <xacro:property name="joint5_origin_rpy" value="${-pi/2} 0 0"/>
+  <xacro:property name="joint5_axis_xyz" value="0 0 1"/>
+  <xacro:property name="joint5_lower_limit" value="${-166*pi/180}"/>
+  <xacro:property name="joint5_upper_limit" value="${166*pi/180}"/>
+  <xacro:property name="joint5_velocity_limit" value="${pi}"/>
+  <xacro:property name="joint5_torque_limit" value="12"/>
+  <xacro:property name="joint5_damping" value="3.0"/>
+  <xacro:property name="joint5_friction" value="0.48"/>
+  <xacro:property name="link5_name" value="link5"/>
+  <xacro:property name="link5_mu" value="0.85"/>
+  <xacro:property name="joint6_name" value="joint6"/>
+  <xacro:property name="joint6_type" value="revolute"/>
+  <xacro:property name="joint6_origin_xyz" value="0 0 0"/>
+  <xacro:property name="joint6_origin_rpy" value="${pi/2} 0 0"/>
+  <xacro:property name="joint6_axis_xyz" value="0 0 1"/>
+  <xacro:property name="joint6_lower_limit" value="${-1/180*pi}"/>
+  <xacro:property name="joint6_upper_limit" value="${215/180*pi}"/>
+  <xacro:property name="joint6_velocity_limit" value="${pi}"/>
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
File: panda_description/urdf/panda_inertial.xacro (robot description, xacro)
@@ -1,76 +1,92 @@
 <?xml version="1.0"?>
+<!-- Macro for inertial properties of Franka Emika Panda -->
 <robot xmlns:xacro="http://www.ros.org/wiki/xacro">
+  <!--            -->
+  <!-- Properties -->
+  <!--            -->
+  <xacro:property name="link0_mesh" value="link0"/>
+  <xacro:property name="link1_mesh" value="link1"/>
+  <xacro:property name="link2_mesh" value="link2"/>
+  <xacro:property name="link3_mesh" value="link3"/>
+  <xacro:property name="link4_mesh" value="link4"/>
+  <xacro:property name="link5_mesh" value="link5"/>
+  <xacro:property name="link6_mesh" value="link6"/>
+  <xacro:property name="link7_mesh" value="link7"/>
+  <xacro:property name="hand_mesh" value="hand"/>
+  <xacro:property name="finger_mesh" value="finger"/>
   <!--       -->
   <!-- Macro -->
   <!--       -->
-  <xacro:macro name="kinova_inertial" params="
-   mesh
+  <xacro:property name="mesh_offset_rpy" value="0 0 0"/>
+  <xacro:macro name="panda_inertial" params="
+    mesh
+    mesh_offset_rpy:=${mesh_offset_rpy}
   ">
-    <xacro:if value="${mesh == 'link0'}">
+    <xacro:if value="${mesh == link0_mesh}">
       <inertial>
-        <origin xyz="-0.025566 -2.87883e-05 0.057332" rpy="0.0 0.0 0.0"/>
+        <origin xyz="-0.025566 -2.87883e-05 0.057332" rpy="${mesh_offset_rpy}"/>
         <mass value="2.814271300104062"/>
         <inertia ixx="0.0075390636364814695" iyy="0.010508017427382959" izz="0.009864933638708275" ixy="-1.5053124574783335e-05" ixz="-0.0012144328835738973" iyz="1.0434803501032979e-05"/>
       </inertial>
     </xacro:if>
-    <xacro:if value="${mesh == 'link1'}">
+    <xacro:if value="${mesh == link1_mesh}">
       <inertial>
-        <origin xyz="-3.72212e-09 -0.0324958 -0.0675818" rpy="0.0 0.0 0.0"/>
+        <origin xyz="-3.72212e-09 -0.0324958 -0.0675818" rpy="${mesh_offset_rpy}"/>
         <mass value="2.6433170427227215"/>
         <inertia ixx="0.017405076982879724" iyy="0.015352077935781732" izz="0.005987891663073857" ixy="-8.687986369621078e-09" ixz="-1.6277819062920423e-08" iyz="0.004510855959102245"/>
       </inertial>
     </xacro:if>
-    <xacro:if value="${mesh == 'link2'}">
+    <xacro:if value="${mesh == link2_mesh}">
       <inertial>
-        <origin xyz="3.17833e-07 -0.06861 0.0322285" rpy="0.0 0.0 0.0"/>
+        <origin xyz="3.17833e-07 -0.06861 0.0322285" rpy="${mesh_offset_rpy}"/>
         <mass value="2.6652755331661186"/>
         <inertia ixx="0.01778694005635383" iyy="0.006044133867952844" izz="0.01571095500455695" ixy="8.70635625879119e-08" ixz="3.752072058394008e-08" iyz="-0.004599490295490376"/>
       </inertial>
     </xacro:if>
-    <xacro:if value="${mesh == 'link3'}">
+    <xacro:if value="${mesh == link3_mesh}">
       <inertial>
-        <origin xyz="0.0469893 0.0316374 -0.031704" rpy="0.0 0.0 0.0"/>
+        <origin xyz="0.0469893 0.0316374 -0.031704" rpy="${mesh_offset_rpy}"/>
         <mass value="2.3293714829045733"/>
         <inertia ixx="0.0075496764161139766" iyy="0.009680676080191398" izz="0.007944557422008086" ixy="-0.0024320464513492225" ixz="-0.003250815048103007" iyz="-0.0021316282421730694"/>
       </inertial>
     </xacro:if>
-    <xacro:if value="${mesh == 'link4'}">
+    <xacro:if value="${mesh == link4_mesh}">
       <inertial>
-        <origin xyz="-0.0360505 0.0337069 0.0319019" rpy="0.0 0.0 0.0"/>
+        <origin xyz="-0.0360505 0.0337069 0.0319019" rpy="${mesh_offset_rpy}"/>
         <mass value="2.3104763646281508"/>
         <inertia ixx="0.007764568814864828" iyy="0.008015776929980149" izz="0.009955882308071066" ixy="0.003371475204045935" ixz="-0.002343621113168248" iyz="0.0022917526161470624"/>
       </inertial>
     </xacro:if>
-    <xacro:if value="${mesh == 'link5'}">
+    <xacro:if value="${mesh == link5_mesh}">
       <inertial>
-        <origin xyz="-6.12525e-06 0.0610427 -0.104176" rpy="0.0 0.0 0.0"/>
+        <origin xyz="-6.12525e-06 0.0610427 -0.104176" rpy="${mesh_offset_rpy}"/>
         <mass value="2.6226426154892004"/>
         <inertia ixx="0.029070538014399377" iyy="0.027638529986528795" izz="0.004251111234400737" ixy="6.208738268725568e-07" ixz="-1.0059151925023392e-05" iyz="-0.007424306477850814"/>
       </inertial>
     </xacro:if>
-    <xacro:if value="${mesh == 'link6'}">
+    <xacro:if value="${mesh == link6_mesh}">
       <inertial>
-        <origin xyz="0.051051 0.00910797 0.0106343" rpy="0.0 0.0 0.0"/>
+        <origin xyz="0.051051 0.00910797 0.0106343" rpy="${mesh_offset_rpy}"/>
         <mass value="1.5025804886626795"/>
         <inertia ixx="0.002940555801469018" iyy="0.00392105201248677" izz="0.0054115603870960195" ixy="-0.00042391108351381507" ixz="0.000610007735338717" iyz="0.00012647545430836214"/>
       </inertial>
     </xacro:if>
-    <xacro:if value="${mesh == 'link7'}">
+    <xacro:if value="${mesh == link7_mesh}">
       <inertial>
-        <origin xyz="0.0109695 0.0107965 0.0650412" rpy="0.0 0.0 0.0"/>
+        <origin xyz="0.0109695 0.0107965 0.0650412" rpy="${mesh_offset_rpy}"/>
         <mass value="0.5237668134788256"/>
         <inertia ixx="0.0008621467959726535" iyy="0.0008613100184801048" izz="0.0006961139396618219" ixy="-0.00011871071570425467" ixz="3.866602604509339e-05" iyz="-9.057841649422724e-05"/>
       </inertial>
     </xacro:if>
-    <xacro:if value="${mesh == 'hand'}">
+    <xacro:if value="${mesh == hand_mesh}">
       <inertial>
-        <origin xyz="-6.7624e-06 0.00152435 0.0275912" rpy="0.0 0.0 0.0"/>
+        <origin xyz="-6.7624e-06 0.00152435 0.0275912" rpy="${mesh_offset_rpy}"/>
         <mass value="0.14060765127978503"/>
         <inertia ixx="0.0005365450414352072" iyy="7.70511954783727e-05" izz="0.0004938176882694914" ixy="1.7911952957732454e-08" ixz="-2.320071910601251e-08" iyz="4.681149945315967e-08"/>
       </inertial>
     </xacro:if>
-    <xacro:if value="${mesh == 'finger'}">
+    <xacro:if value="${mesh == finger_mesh}">
       <inertial>
-        <origin xyz="-6.2561e-06 0.00227781 -0.0277116" rpy="0.0 0.0 0.0"/>
+        <origin xyz="-6.2561e-06 0.00227781 -0.0277116" rpy="${mesh_offset_rpy}"/>
         <mass value="0.2238453537819424"/>
         <inertia ixx="6.74804167363695e-05" iyy="6.627189221641395e-05" izz="1.550396267804825e-05" ixy="-4.1027443646025676e-09" ixz="1.8693673970152995e-08" iyz="1.1967548474390802e-05"/>
