Commit message: Add xacro-based URDF and SDF (with ros2_control)
Signed-off-by: Andrej Orsula <orsula.andrej@gmail.com>

File: panda_description/urdf/panda_utils.xacro (robot description, xacro)
@@ -1,3 +1,4 @@
 <?xml version="1.0"?>
+<!-- Macros for general boilerplate -->
 <robot xmlns:xacro="http://www.ros.org/wiki/xacro">
   <!--                   -->
@@ -8,4 +9,5 @@
   <!-- Macro -->
   <!--       -->
+  <xacro:property name="mesh_offset_rpy" value="0 0 0"/>
   <xacro:macro name="panda_link" params="
     link_name
@@ -13,7 +15,10 @@
     collision:=true
     mu:=1.0
+    mesh_offset_rpy:=${mesh_offset_rpy}
+    gazebo_self_collide:=false
   ">
     <link name="${link_name}">
       <visual>
+        <origin xyz="0 0 0" rpy="${mesh_offset_rpy}"/>
         <geometry>
           <mesh filename="package://panda_description/meshes/visual/${mesh}.dae"/>
@@ -22,4 +27,5 @@
       <xacro:if value="${collision}">
         <collision>
+          <origin xyz="0 0 0" rpy="${mesh_offset_rpy}"/>
           <geometry>
             <mesh filename="package://panda_description/meshes/collision/${mesh}.stl"/>
@@ -27,9 +33,12 @@
         </collision>
       </xacro:if>
-      <xacro:panda_inertial mesh="${mesh}"/>
+      <xacro:panda_inertial mesh="${mesh}" mesh_offset_rpy="${mesh_offset_rpy}"/>
     </link>
     <gazebo reference="${link_name}">
       <mu1 value="${mu}"/>
       <mu2 value="${mu}"/>
+      <xacro:if value="${gazebo_self_collide}">
+        <self_collide>true</self_collide>
+      </xacro:if>
     </gazebo>
   </xacro:macro>
@@ -38,11 +47,11 @@
   <!--       -->
   <xacro:macro name="panda_joint" params="
-    joint_name
-    type
     parent
     child
+    joint_name
+    joint_type
     joint_origin_xyz
     joint_origin_rpy
-    joint_axis_xyz
+    joint_axis_xyz:=unset
     joint_lower_limit:=unset
     joint_upper_limit:=unset
@@ -51,12 +60,18 @@
     joint_damping:=0.0
     joint_friction:=0.0
+    mimic_joint:=none
     safety_limits:=false
     safety_position_margin:=0.0
-    safety_k_position:=100.0
-    safety_k_velocity:=40.0
+    safety_k_position:=0.0
+    safety_k_velocity:=0.0
+    gazebo_spring_stiffness:=0.0
+    gazebo_spring_reference:=0.0
     gazebo_preserve_fixed_joint:=false
   ">
     <!-- Make sure limits are set for non-fixed joints -->
-    <xacro:unless value="${type == 'fixed'}">
+    <xacro:unless value="${joint_type == 'fixed'}">
+      <xacro:if value="${joint_axis_xyz == 'unset'}">
+        <xacro:ERROR_joint_axis_xyz_undefined/>
+      </xacro:if>
       <xacro:if value="${joint_lower_limit == 'unset'}">
         <xacro:ERROR_joint_lower_limit_undefined/>
@@ -72,22 +87,27 @@
       </xacro:if>
     </xacro:unless>
-    <joint name="${joint_name}" type="${type}">
+    <joint name="${joint_name}" type="${joint_type}">
       <parent link="${parent}"/>
       <child link="${child}"/>
       <origin xyz="${joint_origin_xyz}" rpy="${joint_origin_rpy}"/>
-      <axis xyz="${joint_axis_xyz}"/>
-      <xacro:if value="${type == 'revolute' or type == 'prismatic'}">
-        <limit lower="${joint_lower_limit}" upper="${joint_upper_limit}" effort="${joint_torque_limit}" velocity="${joint_velocity_limit}"/>
-      </xacro:if>
-      <xacro:if value="${type == 'continuous'}">
-        <limit effort="${joint_torque_limit}" velocity="${joint_velocity_limit}"/>
-      </xacro:if>
-      <dynamics damping="${joint_damping}" friction="${joint_friction}"/>
-      <xacro:if value="${safety_limits}">
-        <safety_controller soft_lower_limit="${joint_lower_limit+safety_position_margin}" soft_upper_limit="${joint_upper_limit-safety_position_margin}" k_position="${safety_k_position}" k_velocity="${safety_k_velocity}"/>
-      </xacro:if>
+      <xacro:unless value="${joint_type == 'fixed'}">
+        <axis xyz="${joint_axis_xyz}"/>
+        <xacro:if value="${joint_type == 'continuous'}">
+          <limit effort="${joint_torque_limit}" velocity="${joint_velocity_limit}"/>
+        </xacro:if>
+        <xacro:unless value="${joint_type == 'continuous'}">
+          <limit lower="${joint_lower_limit}" upper="${joint_upper_limit}" effort="${joint_torque_limit}" velocity="${joint_velocity_limit}"/>
+        </xacro:unless>
+        <xacro:if value="${safety_limits}">
+          <safety_controller soft_lower_limit="${joint_lower_limit+safety_position_margin}" soft_upper_limit="${joint_upper_limit-safety_position_margin}" k_position="${safety_k_position}" k_velocity="${safety_k_velocity}"/>
+        </xacro:if>
+        <dynamics damping="${joint_damping}" friction="${joint_friction}"/>
+      </xacro:unless>
+      <xacro:unless value="${mimic_joint == 'none'}">
+        <mimic joint="${mimic_joint}"/>
+      </xacro:unless>
     </joint>
     <!-- Transmission for non-fixed joints -->
-    <xacro:unless value="${type == 'fixed'}">
+    <xacro:unless value="${joint_type == 'fixed'}">
       <transmission name="${joint_name}_transmission">
         <type>transmission_interface/SimpleTransmission</type>
@@ -100,6 +120,13 @@
       </transmission>
     </xacro:unless>
+    <!-- Spring stiffness and reference for non-fifex joint -->
+    <xacro:unless value="${joint_type == 'fixed'}">
+      <gazebo reference="${joint_name}">
+        <springStiffness value="${gazebo_spring_stiffness}"/>
+        <springReference value="${gazebo_spring_reference}"/>
+      </gazebo>
+    </xacro:unless>
     <!-- Preserve fixed joint, if desired -->
-    <xacro:if value="${type == 'fixed' and gazebo_preserve_fixed_joint}">
+    <xacro:if value="${joint_type == 'fixed' and gazebo_preserve_fixed_joint}">
       <gazebo reference="${joint_name}">
         <preserveFixedJoint>true</preserveFixedJoint>
@@ -112,11 +139,28 @@
   <!--       -->
   <xacro:macro name="panda_virtual_link" params="
+    parent
     link_name
-    parent
     joint_origin_xyz
     joint_origin_rpy
     gazebo_preserve_fixed_joint:=false
   ">
-    <link name="${link_name}">
+    <xacro:panda_dummy_link
+      name="${link_name}"
+      gazebo_preserve_fixed_joint="${gazebo_preserve_fixed_joint}"
+    />
+    <joint name="${link_name}_virtual_joint" type="fixed">
+      <parent link="${parent}"/>
+      <child link="${link_name}"/>
+      <origin xyz="${joint_origin_xyz}" rpy="${joint_origin_rpy}"/>
+    </joint>
+  </xacro:macro>
+  <!--       -->
+  <!-- Macro -->
+  <!--       -->
+  <xacro:macro name="panda_dummy_link" params="
+    name
+    gazebo_preserve_fixed_joint:=false
+  ">
+    <link name="${name}">
       <xacro:if value="${gazebo_preserve_fixed_joint}">
         <inertial>
@@ -126,9 +170,4 @@
       </xacro:if>
     </link>
-    <joint name="${link_name}_virtual_joint" type="fixed">
-      <parent link="${parent}"/>
-      <child link="${link_name}"/>
-      <origin xyz="${joint_origin_xyz}" rpy="${joint_origin_rpy}"/>
-    </joint>
     <!-- Preserve fixed joint, if desired -->
     <xacro:if value="${gazebo_preserve_fixed_joint}">
