Commit message: Add MoveIt 2 config (integrated with ign_ros2_control)
Signed-off-by: Andrej Orsula <orsula.andrej@gmail.com>

File: panda_description/urdf/panda.urdf (robot description, URDF)
Before this commit: robot panda, 14 links, 13 joints
Joints:
- joint panda_finger_joint2: mimic joint=panda_finger_joint1 -> (none)

File: panda_description/urdf/panda.urdf.xacro (robot description, xacro)
@@ -33,7 +33,7 @@
   <xacro:arg name="ros2_control" default="true"/>
   <!-- The ros2_control plugin that should be loaded for the manipulator ('fake', 'ignition', 'real' or custom) -->
-  <xacro:arg name="ros2_control_plugin" default="fake"/>
+  <xacro:arg name="ros2_control_plugin" default="ignition"/>
   <!-- The output control command interface provided by ros2_control ('position', 'velocity', 'effort' or certain combinations 'position,velocity') -->
-  <xacro:arg name="ros2_control_command_interface" default="position"/>
+  <xacro:arg name="ros2_control_command_interface" default="effort"/>
   <!-- The filepath to parameters of ROS 2 controllers -->
   <xacro:arg name="ros2_controller_parameters" default="$(find panda_moveit_config)/config/controllers_$(arg ros2_control_command_interface).yaml"/>
@@ -45,5 +45,5 @@
   <!-- Prefixes -->
   <xacro:property name="prefix_arm" value="$(arg prefix)"/>
-  <xacro:property name="prefix_hand" value="$(arg prefix)"/>
+  <xacro:property name="prefix_gripper" value="$(arg prefix)"/>
   <!-- Origin of arm in the world -->
   <xacro:property name="world_name" value="world"/>
@@ -81,5 +81,5 @@
     <xacro:panda_gripper
       wrist_flange="${prefix_arm}${wrist_flange_name}"
-      prefix="${prefix_hand}"
+      prefix="${prefix_gripper}"
       origin_xyz="${gripper_offset_xyz}"
       origin_rpy="${gripper_offset_rpy}"

File: panda_description/urdf/panda_gripper.xacro (robot description, xacro)
@@ -23,6 +23,6 @@
   <xacro:property name="joint_finger1_velocity_limit" value="0.2"/>
   <xacro:property name="joint_finger1_torque_limit" value="20"/>
-  <xacro:property name="joint_finger1_damping" value="10.0"/>
-  <xacro:property name="joint_finger1_friction" value="0.5"/>
+  <xacro:property name="joint_finger1_damping" value="0.5"/>
+  <xacro:property name="joint_finger1_friction" value="0.002"/>
   <xacro:property name="link_finger1_name" value="leftfinger"/>
   <xacro:property name="link_finger1_mu" value="1.13"/>
@@ -37,6 +37,6 @@
   <xacro:property name="joint_finger2_velocity_limit" value="0.2"/>
   <xacro:property name="joint_finger2_torque_limit" value="20"/>
-  <xacro:property name="joint_finger2_damping" value="10.0"/>
-  <xacro:property name="joint_finger2_friction" value="0.5"/>
+  <xacro:property name="joint_finger2_damping" value="0.5"/>
+  <xacro:property name="joint_finger2_friction" value="0.002"/>
   <xacro:property name="link_finger2_name" value="rightfinger"/>
   <xacro:property name="link_finger2_mu" value="1.13"/>
@@ -117,5 +117,4 @@
     joint_friction="${joint_finger2_friction}"
     gazebo_preserve_fixed_joint="${gazebo_preserve_fixed_joint}"
-    mimic_joint="${prefix}${joint_finger1_name}"
     />
     <xacro:panda_link

File: panda_moveit_config/srdf/panda.srdf.xacro (robot description, xacro)
@@ -1,43 +1,44 @@
-<?xml version='1.0' encoding='utf-8'?>
-<!--This does not replace URDF, and is not an extension of URDF.
-    This is a format for representing semantic information about the robot structure.
-    A URDF file must exist for this robot as well, where the joints and the links that are referenced are defined
--->
-<robot xmlns:xacro="http://www.ros.org/wiki/xacro" name="panda">
-  <xacro:include filename="$(find moveit_resources_panda_moveit_config)/config/panda_arm.xacro" />
-  <xacro:include filename="$(find moveit_resources_panda_moveit_config)/config/hand.xacro" />
-  <xacro:panda_arm />
-  <xacro:hand />
-  <!--GROUPS: Representation of a set of joints and links. This can be useful for specifying DOF to plan for, defining arms, end effectors, etc-->
-  <!--LINKS: When a link is specified, the parent joint of that link (if it exists) is automatically included-->
-  <!--JOINTS: When a joint is specified, the child link of that joint (which will always exist) is automatically included-->
-  <!--CHAINS: When a chain is specified, all the links along the chain (including endpoints) are included in the group. Additionally, all the joints that are parents to included links are also included. This means that joints along the chain and the parent joint of the base link are included in the group-->
-  <!--SUBGROUPS: Groups can also be formed by referencing to already defined group names-->
-  <group name="panda_arm_hand">
-    <group name="panda_arm" />
-    <group name="hand" />
-  </group>
-  <group_state name="open" group="hand">
-    <joint name="panda_finger_joint1" value="0.035" />
-    <joint name="panda_finger_joint2" value="0.035" />
-  </group_state>
-  <group_state name="close" group="hand">
-    <joint name="panda_finger_joint1" value="0" />
-    <joint name="panda_finger_joint2" value="0" />
-  </group_state>
-  <!--END EFFECTOR: Purpose: Represent information about an end effector.-->
-  <end_effector name="hand" parent_link="panda_link8" group="hand" parent_group="panda_arm" />
-  <!--DISABLE COLLISIONS: By default it is assumed that any link of the robot could potentially come into collision with any other link in the robot. This tag disables collision checking between a specified pair of links. -->
-  <disable_collisions link1="panda_hand" link2="panda_link3" reason="Never" />
-  <disable_collisions link1="panda_hand" link2="panda_link4" reason="Never" />
-  <disable_collisions link1="panda_hand" link2="panda_link6" reason="Never" />
-  <disable_collisions link1="panda_hand" link2="panda_link7" reason="Adjacent" />
-  <disable_collisions link1="panda_leftfinger" link2="panda_link3" reason="Never" />
-  <disable_collisions link1="panda_leftfinger" link2="panda_link4" reason="Never" />
-  <disable_collisions link1="panda_leftfinger" link2="panda_link6" reason="Never" />
-  <disable_collisions link1="panda_leftfinger" link2="panda_link7" reason="Never" />
-  <disable_collisions link1="panda_link3" link2="panda_rightfinger" reason="Never" />
-  <disable_collisions link1="panda_link4" link2="panda_rightfinger" reason="Never" />
-  <disable_collisions link1="panda_link6" link2="panda_rightfinger" reason="Never" />
-  <disable_collisions link1="panda_link7" link2="panda_rightfinger" reason="Never" />
+<?xml version="1.0"?>
+<!-- SRDF for Franka Emika Panda -->
+<robot xmlns:xacro="http://wiki.ros.org/xacro" name="$(arg name)">
+  <!--                   -->
+  <!-- Imported elements -->
+  <!--                   -->
+  <xacro:include filename="$(find panda_moveit_config)/srdf/panda_arm.xacro"/>
+  <xacro:include filename="$(find panda_moveit_config)/srdf/panda_gripper.xacro"/>
+  <!--            -->
+  <!-- Parameters -->
+  <!--            -->
+  <!-- Name of the robot (mandatory) -->
+  <xacro:arg name="name" default="panda"/>
+  <!-- Prefix for all entities -->
+  <xacro:arg name="prefix" default="$(arg name)_"/>
+  <!--            -->
+  <!-- Properties -->
+  <!--            -->
+  <!-- Prefixes -->
+  <xacro:property name="prefix_arm" value="$(arg prefix)"/>
+  <xacro:property name="prefix_gripper" value="$(arg prefix)"/>
+  <!--       -->
+  <!-- Robot -->
+  <!--       -->
+  <xacro:panda_arm
+    prefix="${prefix_arm}"
+  />
+  <xacro:panda_gripper
+    prefix="${prefix_gripper}"
+  />
+  <end_effector group="gripper" name="gripper" parent_group="arm" parent_link="${prefix_arm}hand_tcp"/>
+  <disable_collisions link1="${prefix_gripper}hand" link2="${prefix_arm}link3" reason="Never"/>
+  <disable_collisions link1="${prefix_gripper}hand" link2="${prefix_arm}link4" reason="Never"/>
+  <disable_collisions link1="${prefix_gripper}hand" link2="${prefix_arm}link6" reason="Never"/>
+  <disable_collisions link1="${prefix_gripper}hand" link2="${prefix_arm}link7" reason="Adjacent"/>
+  <disable_collisions link1="${prefix_gripper}leftfinger" link2="${prefix_arm}link3" reason="Never"/>
+  <disable_collisions link1="${prefix_gripper}leftfinger" link2="${prefix_arm}link4" reason="Never"/>
+  <disable_collisions link1="${prefix_gripper}leftfinger" link2="${prefix_arm}link6" reason="Never"/>
+  <disable_collisions link1="${prefix_gripper}leftfinger" link2="${prefix_arm}link7" reason="Never"/>
+  <disable_collisions link1="${prefix_arm}link3" link2="${prefix_gripper}rightfinger" reason="Never"/>
+  <disable_collisions link1="${prefix_arm}link4" link2="${prefix_gripper}rightfinger" reason="Never"/>
+  <disable_collisions link1="${prefix_arm}link6" link2="${prefix_gripper}rightfinger" reason="Never"/>
+  <disable_collisions link1="${prefix_arm}link7" link2="${prefix_gripper}rightfinger" reason="Never"/>
 </robot>

File: panda_moveit_config/srdf/panda_arm.xacro (robot description, xacro)
@@ -1,64 +1,60 @@
-<?xml version="1.0" ?>
-<robot xmlns:xacro="http://www.ros.org/wiki/xacro" name="panda">
-  <xacro:macro name="panda_arm">
-    <!--GROUPS: Representation of a set of joints and links. This can be useful for specifying DOF to plan for, defining arms, end effectors, etc-->
-    <!--LINKS: When a link is specified, the parent joint of that link (if it exists) is automatically included-->
-    <!--JOINTS: When a joint is specified, the child link of that joint (which will always exist) is automatically included-->
-    <!--CHAINS: When a chain is specified, all the links along the chain (including endpoints) are included in the group. Additionally, all the joints that are parents to included links are also included. This means that joints along the chain and the parent joint of the base link are included in the group-->
-    <!--SUBGROUPS: Groups can also be formed by referencing to already defined group names-->
-    <group name="panda_arm">
-      <chain base_link="panda_link0" tip_link="panda_link8" />
+<?xml version="1.0"?>
+<!-- Macro for SRDF of Franka Emika Panda arm -->
+<robot xmlns:xacro="http://wiki.ros.org/xacro">
+  <!--       -->
+  <!-- Macro -->
+  <!--       -->
+  <xacro:macro name="panda_arm" params="
+    prefix:=panda_
+  ">
+    <group name="arm">
+      <chain base_link="${prefix}link0" tip_link="${prefix}hand_tcp"/>
     </group>
-    <!--GROUP STATES: Purpose: Define a named state for a particular group, in terms of joint values. This is useful to define states like 'folded arms'-->
-    <group_state name="ready" group="panda_arm">
-      <joint name="panda_joint1" value="0" />
-      <joint name="panda_joint2" value="-0.785" />
-      <joint name="panda_joint3" value="0" />
-      <joint name="panda_joint4" value="-2.356" />
-      <joint name="panda_joint5" value="0" />
-      <joint name="panda_joint6" value="1.571" />
-      <joint name="panda_joint7" value="0.785" />
+    <group_state group="arm" name="ready">
+      <joint name="${prefix}joint1" value="0"/>
+      <joint name="${prefix}joint2" value="${-pi/4}"/>
+      <joint name="${prefix}joint3" value="0"/>
+      <joint name="${prefix}joint4" value="${-135*pi/180}"/>
+      <joint name="${prefix}joint5" value="0"/>
+      <joint name="${prefix}joint6" value="${pi/2}"/>
+      <joint name="${prefix}joint7" value="${pi/4}"/>
     </group_state>
-    <group_state name="extended" group="panda_arm">
-      <joint name="panda_joint1" value="0" />
-      <joint name="panda_joint2" value="0" />
-      <joint name="panda_joint3" value="0" />
-      <joint name="panda_joint4" value="0" />
-      <joint name="panda_joint5" value="0" />
-      <joint name="panda_joint6" value="1.571" />
-      <joint name="panda_joint7" value="0.785" />
+    <group_state group="arm" name="extended">
+      <joint name="${prefix}joint1" value="0"/>
+      <joint name="${prefix}joint2" value="0"/>
+      <joint name="${prefix}joint3" value="0"/>
+      <joint name="${prefix}joint4" value="0"/>
+      <joint name="${prefix}joint5" value="0"/>
+      <joint name="${prefix}joint6" value="${pi/2}"/>
+      <joint name="${prefix}joint7" value="${pi/4}"/>
     </group_state>
-    <group_state name="transport" group="panda_arm">
-      <joint name="panda_joint1" value="0" />
-      <joint name="panda_joint2" value="-0.5599" />
-      <joint name="panda_joint3" value="0" />
-      <joint name="panda_joint4" value="-2.97" />
-      <joint name="panda_joint5" value="0" />
-      <joint name="panda_joint6" value="0" />
-      <joint name="panda_joint7" value="0.785" />
+    <group_state group="arm" name="transport">
+      <joint name="${prefix}joint1" value="0"/>
+      <joint name="${prefix}joint2" value="${-32.08*pi/180}"/>
+      <joint name="${prefix}joint3" value="0"/>
+      <joint name="${prefix}joint4" value="${-170.17*pi/180}"/>
+      <joint name="${prefix}joint5" value="0"/>
+      <joint name="${prefix}joint6" value="0"/>
+      <joint name="${prefix}joint7" value="${pi/4}"/>
     </group_state>
-    <!--END EFFECTOR: Purpose: Represent information about an end effector.-->
-    <!--VIRTUAL JOINT: Purpose: this element defines a virtual joint between a robot link and an external frame of reference (considered fixed with respect to the robot)-->
-    <virtual_joint name="virtual_joint" type="floating" parent_frame="world" child_link="panda_link0" />
-    <!--DISABLE COLLISIONS: By default it is assumed that any link of the robot could potentially come into collision with any other link in the robot. This tag disables collision checking between a specified pair of links. -->
-    <disable_collisions link1="panda_link0" link2="panda_link1" reason="Adjacent" />
-    <disable_collisions link1="panda_link0" link2="panda_link2" reason="Never" />
-    <disable_collisions link1="panda_link0" link2="panda_link3" reason="Never" />
-    <disable_collisions link1="panda_link0" link2="panda_link4" reason="Never" />
-    <disable_collisions link1="panda_link1" link2="panda_link2" reason="Adjacent" />
-    <disable_collisions link1="panda_link1" link2="panda_link3" reason="Never" />
-    <disable_collisions link1="panda_link1" link2="panda_link4" reason="Never" />
-    <disable_collisions link1="panda_link2" link2="panda_link3" reason="Adjacent" />
-    <disable_collisions link1="panda_link2" link2="panda_link4" reason="Never" />
-    <disable_collisions link1="panda_link2" link2="panda_link6" reason="Never" />
-    <disable_collisions link1="panda_link3" link2="panda_link4" reason="Adjacent" />
-    <disable_collisions link1="panda_link3" link2="panda_link5" reason="Never" />
-    <disable_collisions link1="panda_link3" link2="panda_link6" reason="Never" />
-    <disable_collisions link1="panda_link3" link2="panda_link7" reason="Never" />
-    <disable_collisions link1="panda_link4" link2="panda_link5" reason="Adjacent" />
-    <disable_collisions link1="panda_link4" link2="panda_link6" reason="Never" />
-    <disable_collisions link1="panda_link4" link2="panda_link7" reason="Never" />
-    <disable_collisions link1="panda_link5" link2="panda_link6" reason="Adjacent" />
-    <disable_collisions link1="panda_link6" link2="panda_link7" reason="Adjacent" />
+    <disable_collisions link1="${prefix}link0" link2="${prefix}link1" reason="Adjacent"/>
+    <disable_collisions link1="${prefix}link0" link2="${prefix}link2" reason="Never"/>
+    <disable_collisions link1="${prefix}link0" link2="${prefix}link3" reason="Never"/>
+    <disable_collisions link1="${prefix}link0" link2="${prefix}link4" reason="Never"/>
+    <disable_collisions link1="${prefix}link1" link2="${prefix}link2" reason="Adjacent"/>
+    <disable_collisions link1="${prefix}link1" link2="${prefix}link3" reason="Never"/>
+    <disable_collisions link1="${prefix}link1" link2="${prefix}link4" reason="Never"/>
+    <disable_collisions link1="${prefix}link2" link2="${prefix}link3" reason="Adjacent"/>
+    <disable_collisions link1="${prefix}link2" link2="${prefix}link4" reason="Never"/>
+    <disable_collisions link1="${prefix}link2" link2="${prefix}link6" reason="Never"/>
+    <disable_collisions link1="${prefix}link3" link2="${prefix}link4" reason="Adjacent"/>
+    <disable_collisions link1="${prefix}link3" link2="${prefix}link5" reason="Never"/>
+    <disable_collisions link1="${prefix}link3" link2="${prefix}link6" reason="Never"/>
+    <disable_collisions link1="${prefix}link3" link2="${prefix}link7" reason="Never"/>
+    <disable_collisions link1="${prefix}link4" link2="${prefix}link5" reason="Adjacent"/>
+    <disable_collisions link1="${prefix}link4" link2="${prefix}link6" reason="Never"/>
+    <disable_collisions link1="${prefix}link4" link2="${prefix}link7" reason="Never"/>
+    <disable_collisions link1="${prefix}link5" link2="${prefix}link6" reason="Adjacent"/>
+    <disable_collisions link1="${prefix}link6" link2="${prefix}link7" reason="Adjacent"/>
   </xacro:macro>
 </robot>
