Commit message: Tune PIDs gains v1 (quick manual approach)
Signed-off-by: Andrej Orsula <orsula.andrej@gmail.com>

File: panda_description/urdf/panda_gripper.xacro (robot description, xacro)
@@ -23,6 +23,6 @@
   <xacro:property name="joint_finger1_velocity_limit" value="0.2"/>
   <xacro:property name="joint_finger1_torque_limit" value="20"/>
-  <xacro:property name="joint_finger1_damping" value="0.5"/>
-  <xacro:property name="joint_finger1_friction" value="0.002"/>
+  <xacro:property name="joint_finger1_damping" value="3.0"/>
+  <xacro:property name="joint_finger1_friction" value="0.4"/>
   <xacro:property name="link_finger1_name" value="leftfinger"/>
   <xacro:property name="link_finger1_mu" value="1.13"/>
@@ -37,6 +37,6 @@
   <xacro:property name="joint_finger2_velocity_limit" value="0.2"/>
   <xacro:property name="joint_finger2_torque_limit" value="20"/>
-  <xacro:property name="joint_finger2_damping" value="0.5"/>
-  <xacro:property name="joint_finger2_friction" value="0.002"/>
+  <xacro:property name="joint_finger2_damping" value="3.0"/>
+  <xacro:property name="joint_finger2_friction" value="0.4"/>
   <xacro:property name="link_finger2_name" value="rightfinger"/>
   <xacro:property name="link_finger2_mu" value="1.13"/>
