Commit message: Fix URDF xacro for `panda_dummy_link`
Signed-off-by: Andrej Orsula <orsula.andrej@gmail.com>

File: panda_description/urdf/panda.urdf.xacro (robot description, xacro)
@@ -58,5 +58,5 @@
   <!-- Dummy world link that the robot is fixed to -->
   <xacro:panda_dummy_link
-    name="${world_name}"
+    link_name="${world_name}"
     gazebo_preserve_fixed_joint="$(arg gazebo_preserve_fixed_joint)"
   />

File: panda_description/urdf/panda_utils.xacro (robot description, xacro)
@@ -146,5 +146,5 @@
   ">
     <xacro:panda_dummy_link
-      name="${link_name}"
+      link_name="${link_name}"
       gazebo_preserve_fixed_joint="${gazebo_preserve_fixed_joint}"
     />
@@ -159,8 +159,8 @@
   <!--       -->
   <xacro:macro name="panda_dummy_link" params="
-    name
+    link_name
     gazebo_preserve_fixed_joint:=false
   ">
-    <link name="${name}">
+    <link name="${link_name}">
       <xacro:if value="${gazebo_preserve_fixed_joint}">
         <inertial>
